File: placebo.kicad_pcb (KiCad board)
At the start: 2 copper layers, 19 x 29.2 mm, 13 parts, among them J1 ExtPower, J2 TagConnect, J3 Conn_01x10, J4 Conn_01x10, U1 AP7370-33W5-7, U2 STM32G0xxFx

Commit message: update docs
Parts:
- added REF**: OSHW-Logo2_7.3x6mm_Copper, Symbol:OSHW-Logo2_7.3x6mm_Copper, B.Cu at (74.2, 94.7)

Commit message: rev 2
Parts:
- removed the REF** at (74.2, 94.7)
- added REF**: OSHW-Logo_5.7x6mm_SilkScreen, Symbol:OSHW-Logo_5.7x6mm_SilkScreen, B.Cu at (74.3, 90.0)
- moved G*** 1.14 mm to (71.2, 86.2)
- moved J2 0.81 mm to (74.8, 84.3), turned to 0 degrees
- turned C2 to -90 degrees
Routing:
- net GND: track 22.5 -> 12.3 mm, vias 4 -> 6
- net +3V3: track 35.7 -> 29.6 mm, vias 1 -> 2
- net /SwdIO: track 20.3 -> 25.0 mm, vias 1 -> 0
- net /SwdClk: track 21.5 -> 19.4 mm
- net /PB9: track 12.0 -> 11.1 mm
Other:
- board size 19 x 29.2 mm -> 19.1 x 29.2 mm
- board text added: "STM32G0xxFx breakout rev. 0x2"
- board text added: "swdclk"
- board text added: "swdio"
- board text removed: "-"
- board text removed: "10"
- board text removed: "11"
- board text removed: "STM32G0xxFx breakout"

Commit message: rev 0x3
Parts:
- J1: footprint Connector_PinHeader_2.54mm:PinHeader_1x03_P2.54mm_Vertical -> Connector_PinHeader_2.54mm:PinHeader_1x05_P2.54mm_Vertical
- moved J1 2.55 mm to (69.2, 108.7)
Connections:
- J1 pad 2: Net-(C1-Pad1) -> GND
- J1 pad 3: Net-(C1-Pad1) -> GND
Routing:
- net GND: track 12.3 -> 14.1 mm, vias 6 -> 5
- net /nRST: track 20.7 -> 20.2 mm
Other:
- outline, holes or cut-outs redrawn
- board text added: "STM32G0xxFx breakout rev. 0x3"
- board text removed: "GND VBAT"
- board text removed: "STM32G0xxFx breakout rev. 0x2"

Commit message: rev 0x4
Other:
- board text added: "STM32G0xxFx breakout rev. 0x4"
- board text removed: "STM32G0xxFx breakout rev. 0x3"

Commit message: PlaceboConnect
Parts:
- removed J1: ExtPower, Connector_PinHeader_2.54mm:PinHeader_1x05_P2.54mm_Vertical
- removed J3, J4: Conn_01x10, Connector_PinHeader_2.54mm:PinHeader_1x10_P2.54mm_Vertical
- removed the REF** at (74.3, 90.0)
- added D1: DNP, LED_SMD:LED_0603_1608Metric, F.Cu at (72.8, 104.4)
- added R2: DNP, Resistor_SMD:R_0603_1608Metric, F.Cu at (75.9, 104.4)
- added R3: DNP, Resistor_SMD:R_0603_1608Metric, F.Cu at (75.9, 106.0)
- added REF**: OSHW-Logo2_7.3x6mm_SilkScreen, Symbol:OSHW-Logo2_7.3x6mm_SilkScreen, B.Cu at (74.3, 90.0)
- added U3: PlaceboConnect, placebo:PlaceboConnect, F.Cu at (74.4, 94.7)
- moved G*** 1.61 mm to (69.6, 85.9)
- moved J2 0.57 mm to (74.3, 84.6)
Connections:
- net Net-(C1-Pad1) renamed VCC
Routing:
- net /PB3: track 11.1 -> 26.9 mm
- net GND: track 13.9 -> 20.8 mm
- net Net-(D1-K): track 0.00 -> 3.21 mm
- net VCC: track 11.8 -> 14.5 mm
- net /PB7: track 10.4 -> 12.9 mm
- net /SwdIO: track 24.8 -> 22.3 mm, vias 0 -> 1
- net +3V3: track 28.9 -> 31.1 mm
- net /SwdClk: track 19.3 -> 19.8 mm
- net /PB9: vias 1 -> 0
Other:
- board size 19.1 x 29.2 mm -> 19.1 x 29.1 mm
- board text added: "STM32G0xxFx Breakout rev. 0x5"
- board text removed: "1"
- board text removed: "20"
- board text removed: "STM32G0xxFx breakout rev. 0x4"
- board text removed: "◢◤"

Commit message: PlaceboConnect-cutout
Parts:
- U3: footprint placebo:PlaceboConnect -> placebo:PlaceboConnect_Cutout
- renumbered G*** to LOGO1
Changed lines of the file:
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@@
       (layer "F.SilkS" (type "Top Silk Screen") (color "White"))
       (layer "F.Paste" (type "Top Solder Paste"))
-      (layer "F.Mask" (type "Top Solder Mask") (color "#000000B3") (thickness 0.0254))
+      (layer "F.Mask" (type "Top Solder Mask") (color "#0000004A") (thickness 0.0254))
       (layer "F.Cu" (type "copper") (thickness 0.0356))
       (layer "dielectric 1" (type "prepreg") (color "#000000FF") (thickness 0.1702) (material "FR408-HR") (epsilon_r 3.7) (loss_tangent 0.0091))
       (layer "B.Cu" (type "copper") (thickness 0.0356))
-      (layer "B.Mask" (type "Bottom Solder Mask") (color "#000000B3") (thickness 0.0254))
+      (layer "B.Mask" (type "Bottom Solder Mask") (color "#0000004D") (thickness 0.0254))
       (layer "B.Paste" (type "Bottom Solder Paste"))
       (layer "B.SilkS" (type "Bottom Silk Screen") (color "White"))
@@
   (net 24 "Net-(D1-K)")
   (net 25 "VCC")
-  (footprint "placebo:PlaceboConnect" locked (layer "F.Cu")
+  (footprint "placebo:PlaceboConnect_Cutout" locked (layer "F.Cu")
     (at 74.422 94.742)
     (property "Sheetfile" "File: placebo.kicad_sch")
     (property "Sheetname" "")
     (attr through_hole)
-    (fp_text reference "U3" (at -0.0508 -14.351 unlocked) (layer "F.SilkS") hide
-        (effects (font (size 1 1) (thickness 0.15)))
-    )
-    (fp_text value "PlaceboConnect" (at 0.1778 -15.8242 unlocked) (layer "F.Fab")
-        (effects (font (size 1 1) (thickness 0.15)))
-    )
-    (fp_text user "${REFERENCE}" (at 0 17.2974 unlocked) (layer "F.Fab")
-        (effects (font (size 1 1) (thickness 0.15)))
-    )
-    (fp_line (start -9.728132 -11.432918) (end -9.728132 11.50963)
-      (stroke (width 0.1) (type default)) (layer "Edge.Cuts"))
-    (fp_line (start -6.9862 14.303567) (end -6.9862 14.83062)
-      (stroke (width 0.1) (type default)) (layer "Edge.Cuts"))
-    (fp_line (start -5.971468 15.897357) (end 5.787982 15.897483)
-      (stroke (width 0.1) (type default)) (layer "Edge.Cuts"))
-    (fp_line (start 6.860862 14.359973) (end 6.854782 14.881943)
+    (fp_text reference "U3" (at 0.254 0 unlocked) (layer "F.SilkS") hide
+        (effects (font (size 1 1) (thickness 0.15)))
+    )
+    (fp_text value "PlaceboConnect" (at 0 -14.097 unlocked) (layer "F.Fab")
+        (effects (font (size 1 1) (thickness 0.15)))
+    )
+    (fp_text user "${REFERENCE}" (at -0.127 17.2974 unlocked) (layer "F.Fab")
+        (effects (font (size 1 1) (thickness 0.15)))
+    )
+    (fp_line (start -9.728132 -11.43) (end -9.728132 11.506049)
+      (stroke (width 0.1) (type default)) (layer "Edge.Cuts"))
+    (fp_line (start -6.985 14.299986) (end -6.9862 14.83062)
+      (stroke (width 0.1) (type default)) (layer "Edge.Cuts"))
+    (fp_line (start -5.971468 15.897357) (end 5.763767 15.896675)
+      (stroke (width 0.1) (type default)) (layer "Edge.Cuts"))
+    (fp_line (start 6.830504 14.3256) (end 6.830504 14.881943)
       (stroke (width 0.1) (type default)) (layer "Edge.Cuts"))
     (fp_line (start 7.643353 -13.160118) (end -8.000932 -13.160118)
       (stroke (width 0.1) (type default)) (layer "Edge.Cuts"))
-    (fp_line (start 9.370553 -11.432918) (end 9.37049 11.612038)
-      (stroke (width 0.1) (type default)) (layer "Edge.Cuts"))
-    (fp_arc (start -9.728132 -11.432918) (mid -9.222246 -12.654232) (end -8.000932 -13.160118)
-      (stroke (width 0.1) (type default)) (layer "Edge.Cuts"))
-    (fp_arc (start -8.000932 13.23683) (mid -9.222247 12.730945) (end -9.728132 11.50963)
-      (stroke (width 0.1) (type default)) (layer "Edge.Cuts"))
-    (fp_arc (start -8.000932 13.23683) (mid -7.264792 13.552578) (end -6.9862 14.303567)
-      (stroke (width 0.1) (type default)) (layer "Edge.Cuts"))
-    (fp_arc (start -5.971468 15.897357) (mid -6.707608 15.581609) (end -6.9862 14.83062)
-      (stroke (width 0.1) (type default)) (layer "Edge.Cuts"))
-    (fp_arc (start 6.854782 14.881943) (mid 6.539059 15.618377) (end 5.787982 15.897483)
-      (stroke (width 0.1) (type default)) (layer "Edge.Cuts"))
-    (fp_arc (start 6.860862 14.359973) (mid 7.111067 13.666034) (end 7.7724 13.339238)
-      (stroke (width 0.1) (type default)) (layer "Edge.Cuts"))
-    (fp_arc (start 7.643353 -13.160118) (mid 8.864668 -12.654235) (end 9.370553 -11.432918)
-      (stroke (width 0.1) (type default)) (layer "Edge.Cuts"))
-    (fp_arc (start 9.37049 11.612038) (mid 8.909673 12.788582) (end 7.7724 13.339238)
+    (fp_line (start 9.370553 -11.432918) (end 9.37049 11.608457)
+      (stroke (width 0.1) (type default)) (layer "Edge.Cuts"))
+    (fp_arc (start -9.728132 -11.43) (mid -9.223279 -12.653201) (end -8.000932 -13.160118)
+      (stroke (width 0.1) (type default)) (layer "Edge.Cuts"))
+    (fp_arc (start -8.001 13.233249) (mid -9.222269 12.727338) (end -9.728132 11.506049)
+      (stroke (width 0.1) (type default)) (layer "Edge.Cuts"))
+    (fp_arc (start -8.000932 13.233249) (mid -7.264378 13.548916) (end -6.985 14.299986)
+      (stroke (width 0.1) (type default)) (layer "Edge.Cuts"))
+    (fp_arc (start -5.971468 15.897357) (mid -6.707607 15.581609) (end -6.9862 14.83062)
+      (stroke (width 0.1) (type default)) (layer "Edge.Cuts"))
+    (fp_arc (start 6.830504 14.3256) (mid 7.101764 13.6573) (end 7.747 13.335)
+      (stroke (width 0.1) (type default)) (layer "Edge.Cuts"))
+    (fp_arc (start 6.830504 14.881943) (mid 6.514753 15.61808) (end 5.763767 15.896675)
+      (stroke (width 0.1) (type default)) (layer "Edge.Cuts"))
+    (fp_arc (start 7.643353 -13.160118) (mid 8.864665 -12.654232) (end 9.370553 -11.432918)
+      (stroke (width 0.1) (type default)) (layer "Edge.Cuts"))
+    (fp_arc (start 9.37049 11.608457) (mid 8.900859 12.793422) (end 7.747 13.335)
       (stroke (width 0.1) (type default)) (layer "Edge.Cuts"))
     (pad "1" thru_hole circle locked (at -7.767 -11.41 180) (size 1.7 1.7) (drill 1) (layers *.Cu *.Mask)
@@
     )
   )
-  (footprint "LOGO" (layer "F.Cu")
+  (footprint "LOGO" locked (layer "F.Cu")
     (at 69.596 85.852 8)
     (attr board_only exclude_from_pos_files exclude_from_bom)
-    (fp_text reference "G***" (at 0 0 8) (layer "F.SilkS") hide
+    (fp_text reference "LOGO1" (at 0 0 8) (layer "F.SilkS") hide
         (effects (font (size 1.524 1.524) (thickness 0.3)))
     )
