File: placebo.kicad_pcb (KiCad board)
At the start: 2 copper layers, 19.1 x 29.1 mm, 19 parts, among them J2 TagConnect, U1 AP7370-33W5-7, U2 STM32G0xxFx, U3 PlaceboConnect

Commit message: rev.0x7
Parts:
- removed kibuzzard-62FAD1FB: G***, kibuzzard-62FAD1FB
- removed kibuzzard-62FAD239: G***, kibuzzard-62FAD239
Connections:
- net /UartRx renamed /PA3
- net /UartTx renamed /PA2
Other:
- board text added: "Placebo Proto Board rev. 0x7"
- board text removed: "STM32G0xxFx Proto Board rev. 0x6"

Commit message: rev. 0x8
Parts:
- added kibuzzard-631021FD: G***, kibuzzard-631021FD, F.Cu at (74.1, 106.7)
- moved R2 3.41 mm to (71.3, 105.0), turned to 0 degrees
- moved R3 0.82 mm to (74.5, 105.0)
- moved LOGO1 0.61 mm to (69.1, 84.2)
- moved R4 0.58 mm to (77.7, 105.0), turned to 180 degrees
- moved D1 0.54 mm to (69.3, 108.7)
- moved FID1 0.36 mm to (76.2, 88.4)
Connections:
- R2 pad 1: /PB3 -> /PC15
Routing:
- net /PC15: track 8.00 -> 33.6 mm
- net /PB3: track 25.9 -> 11.1 mm
- net VCC: track 18.9 -> 15.3 mm
- net GND: track 20.3 -> 19.5 mm, vias 5 -> 6
- net Net-(U1-NC): track 6.93 -> 7.62 mm
- net Net-(D1-K): track 7.82 -> 7.14 mm
Other:
- board text added: "Placebo Proto Board rev. 0x8"
- board text removed: "Placebo Proto Board rev. 0x7"
- board text removed: "swdclk"
- board text removed: "swdio"
