File: placebo.kicad_pcb (KiCad board)
At the start: 2 copper layers, 19.1 x 29.1 mm, 18 parts, among them J2 TagConnect, U1 AP7370-33W5-7, U2 STM32G0xxFx, U3 PlaceboConnect

Commit message: panel rev. 0x8
Parts:
- moved FID1 2.26 mm to (78.1, 87.2)
Changed lines of the file:
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@@
     (fp_arc (start 6.830504 14.881943) (mid 6.514753 15.61808) (end 5.763767 15.896675)
       (stroke (width 0.1) (type default)) (layer "Edge.Cuts"))
-    (fp_arc (start 7.643353 -13.160118) (mid 8.864665 -12.654232) (end 9.370553 -11.432918)
+    (fp_arc (start 7.643353 -13.160118) (mid 8.864669 -12.654232) (end 9.370553 -11.432918)
       (stroke (width 0.1) (type default)) (layer "Edge.Cuts"))
     (fp_arc (start 9.37049 11.608457) (mid 8.900859 12.793422) (end 7.747 13.335)
@@
   )
   (footprint "Fiducial:Fiducial_0.5mm_Mask1.5mm" (layer "F.Cu")
-    (at 76.1746 88.4174)
+    (at 78.105 87.249)
     (descr "Circular Fiducial, 0.5mm bare copper, 1.5mm soldermask opening")
     (tags "fiducial")

Commit message: update BOM
Parts:
- C1, C2: value 1uF -> 10uF
- D1: value DNP -> SML-D12W8WT86A
- R2: value DNP -> 470R
Changed lines of the file:
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@@
         (effects (font (size 0.6 0.6) (thickness 0.15)))
     )
-    (fp_text value "1uF" (at 0 1.43 90) (layer "F.Fab")
+    (fp_text value "10uF" (at 0 1.43 90) (layer "F.Fab")
         (effects (font (size 1 1) (thickness 0.15)))
     )
@@
         (effects (font (size 0.6 0.6) (thickness 0.15)))
     )
-    (fp_text value "DNP" (at 0 1.43) (layer "F.Fab")
+    (fp_text value "470R" (at 0 1.43) (layer "F.Fab")
         (effects (font (size 1 1) (thickness 0.15)))
     )
@@
         (effects (font (size 0.6 0.6) (thickness 0.15)))
     )
-    (fp_text value "1uF" (at 0 1.43 90) (layer "F.Fab")
+    (fp_text value "10uF" (at 0 1.43 90) (layer "F.Fab")
         (effects (font (size 1 1) (thickness 0.15)))
     )
@@
         (effects (font (size 0.6 0.6) (thickness 0.15)))
     )
-    (fp_text value "DNP" (at 0 1.43 90) (layer "F.Fab")
-        (effects (font (size 1 1) (thickness 0.15)))
-    )
+    (fp_text value "SML-D12W8WT86A" (at 0 1.43 90) (layer "F.Fab")
+        (effects (font (size 1 1) (thickness 0.15)))
+    )
