File: placebo-panel.kicad_pcb (KiCad board)
At the start: 2 copper layers, 0 parts

Commit message: rev.0x6
Parts:
- added ?: , , F.Cu at (0.00, 0.00)
- added C1: 1uF, Capacitor_SMD:C_0603_1608Metric, F.Cu at (99.0, 54.2)
- added C2: 1uF, Capacitor_SMD:C_0603_1608Metric, F.Cu at (90.8, 54.2)
- added C3: 100nF, Capacitor_SMD:C_0603_1608Metric, F.Cu at (89.8, 43.8)
- added C4: 10uF, Capacitor_SMD:C_0603_1608Metric, F.Cu at (89.8, 46.9)
- added C5: 100nF, Capacitor_SMD:C_0603_1608Metric, F.Cu at (97.9, 43.1)
- added D1: DNP, LED_SMD:LED_0603_1608Metric, F.Cu at (89.7, 61.0)
- added FID1: Fiducial, Fiducial:Fiducial_0.5mm_Mask1.5mm, F.Cu at (96.4, 41.2)
- added FID1000: Fiducial_0.75mm_Mask2.25mm, Fiducial:Fiducial_0.75mm_Mask2.25mm, F.Cu at (80.0, 30.0)
- added J2: TagConnect, placebo:Tag-Connect_TC2030-IDC-NL_2x03_P1.27mm_Vertical, F.Cu at (94.9, 37.4)
- added LOGO1: LOGO, LOGO, F.Cu at (89.8, 36.3)
- added R1: 10K, Resistor_SMD:R_0603_1608Metric, F.Cu at (94.9, 43.1)
- added R2: DNP, Resistor_SMD:R_0603_1608Metric, F.Cu at (95.2, 56.9)
- added R3: DNP, Resistor_SMD:R_0603_1608Metric, F.Cu at (95.2, 58.6)
- added R4: DNP, Resistor_SMD:R_0603_1608Metric, F.Cu at (97.7, 57.7)
- added REF**: Mousebite, placebo:Mousebite, F.Cu at (93.3, 32.9)
- added REF**: Mousebite, placebo:Mousebite, F.Cu at (84.0, 42.4)
- added REF**: Fiducial_0.75mm_Mask2.25mm, Fiducial:Fiducial_0.75mm_Mask2.25mm, F.Cu at (242.0, 30.0)
- added REF**: Mousebite, placebo:Mousebite, F.Cu at (84.0, 55.1)
- added REF**: Fiducial_0.75mm_Mask2.25mm, Fiducial:Fiducial_0.75mm_Mask2.25mm, F.Cu at (80.0, 260.0)
- added REF**: OSHW-Logo2_7.3x6mm_SilkScreen, Symbol:OSHW-Logo2_7.3x6mm_SilkScreen, B.Cu at (94.9, 42.8)
- added U1: AP7370-33W5-7, Package_TO_SOT_SMD:TSOT-23-5_HandSoldering, F.Cu at (94.9, 54.1)
- added U2: STM32G0xxFx, Package_SO:TSSOP-20_4.4x6.5mm_P0.65mm, F.Cu at (94.9, 47.5)
- added U3: PlaceboConnect, placebo:PlaceboConnect_Cutout, F.Cu at (95.0, 47.5)
- added kibuzzard-62FAD1FB: G***, kibuzzard-62FAD1FB, F.Cu at (89.7, 56.7)
- added kibuzzard-62FAD239: G***, kibuzzard-62FAD239, F.Cu at (89.7, 58.6)
Routing:
- net (no net): track 0.00 -> 291.6 mm, vias 0 -> 9
- added copper zone on B.Cu, net (none)
Other:
- board outline added: 167.9 x 238 mm
- board text added: "21.78 31.7"
- board text added: "STM32G0xxFx Proto Board rev. 0x6"
- board text added: "swdclk"
- board text added: "swdio"
- board text added: "vitaly.codes/placebo"
