File: placebo.kicad_sch (KiCad schematic)
At the start: 12 parts, among them J1 ExtPower, J2 TagConnect, J3 Conn_01x10, J4 Conn_01x10, U1 AP7370-33W5-7, U2 STM32G0xxFx

Commit message: rev 0x3
Parts:
- J1: footprint Connector_PinHeader_2.54mm:PinHeader_1x03_P2.54mm_Vertical -> Connector_PinHeader_2.54mm:PinHeader_1x05_P2.54mm_Vertical; symbol Connector_Generic:Conn_01x03 -> Connector_Generic:Conn_01x05
Connections:
- net GND: now also J1.2 (Pin_2), J1.3 (Pin_3)
- net at C1.1, U1.1 (VIN): now also J1.4 (Pin_4), J1.5 (Pin_5); no longer J1.2 (Pin_2), J1.3 (Pin_3)

Commit message: rev 0x4
Parts:
- U: renamed from C1; value 1uF -> (none); footprint Capacitor_SMD:C_0603_1608Metric -> (none)
- U: renamed from U1; value AP7370-33W5-7 -> (none); footprint Package_TO_SOT_SMD:TSOT-23-5_HandSoldering -> (none)
- U: renamed from J2; value TagConnect -> (none); footprint placebo:Tag-Connect_TC2030-IDC-NL_2x03_P1.27mm_Vertical -> (none)
- U: renamed from C5; value 100nF -> (none); footprint Capacitor_SMD:C_0603_1608Metric -> (none)
- U: renamed from J3; value Conn_01x10 -> (none); footprint Connector_PinHeader_2.54mm:PinHeader_1x10_P2.54mm_Vertical -> (none)
- U: renamed from C2; value 1uF -> (none); footprint Capacitor_SMD:C_0603_1608Metric -> (none)
- U: renamed from J4; value Conn_01x10 -> (none); footprint Connector_PinHeader_2.54mm:PinHeader_1x10_P2.54mm_Vertical -> (none)
- U: renamed from J1; value ExtPower -> (none); footprint Connector_PinHeader_2.54mm:PinHeader_1x05_P2.54mm_Vertical -> (none)
- U: renamed from R1; value 10K -> (none); footprint Resistor_SMD:R_0603_1608Metric -> (none)
- U: renamed from C4; value 10uF -> (none); footprint Capacitor_SMD:C_0603_1608Metric -> (none)
- U: renamed from U2; value STM32G0xxFx -> (none); footprint Package_SO:TSSOP-20_4.4x6.5mm_P0.65mm -> (none)
- U: renamed from C3; value 100nF -> (none); footprint Capacitor_SMD:C_0603_1608Metric -> (none)

Commit message: PlaceboConnect
Parts:
- removed U (x2): (no value), symbol Connector_Generic:Conn_01x10
- removed U: (no value), symbol Connector_Generic:Conn_01x05
- added D: LED, symbol Device:LED
- added U (x2): (no value), symbol Device:R
- added U: PlaceboConnect, placebo:PlaceboConnect, symbol Placebo:PlaceboConnect
Connections:
- net +3V3: now also D.2 (A), U.4 (VDD)
- net GND: now also U.2, U.21 (GND), U.22 (GND), U.5 (GND)
- net PA0: now also U.7 (PA0)
- net PA1: now also U.8 (PA1)
- net PA11: now also U.16 (PA11)
- net PA12: now also U.17 (PA12)
- net PA4: now also U.11 (PA4)
- net PA5: now also U.12 (PA5)
- net PA6: now also U.13 (PA6)
- net PA7: now also U.14 (PA7)
- net PB0: now also U.15 (PB0)
- net PB3: now also U.1, U.20 (PB3)
- net PB7: now also U.1 (PB7)
- net PB9: now also U.2 (PB9)
- net PC15: now also U.3 (PC15)
- net SwdClk: now also U.19 (PA14)
- net SwdIO: now also U.18 (PA13)
- net UartRx: now also U.10 (PA3)
- net UartTx: now also U.9 (PA2)
- net nRST: now also U.6 (~RESET)
- net VCC: now reaches U.1, U.1 (VIN)
- net VCC: now also U.23 (VBAT), U.24 (VBAT)
- new net: D.1 (K), U.1, U.2
Other:
- moved on the sheet: U

Commit message: rev. 0x6
Parts:
- added U: (no value), symbol Device:R
Connections:
- net VCC: now also U.1
- net at U.3 (NC): now also U.2
Other:
- moved on the sheet: D, U

Commit message: panel
Changed lines of the file:
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@@
     (stroke (width 0) (type solid))
   )
-  (wire (pts (xy 86.36 96.52) (xy 86.36 97.155))
+  (wire (pts (xy 86.36 96.52) (xy 86.36 102.87))
     (stroke (width 0) (type solid))
   )
@@
     (pin "2")
   )
-  (symbol (lib_id "power:GND") (at 86.36 97.155 0) (unit 1)
-    (in_bom yes) (on_board yes)
-    (default_instance (reference "U") (unit 1) (value "") (footprint ""))
-    (property "Reference" "U" (id 0) (at 86.36 103.505 0)
-      (effects (font (size 1.27 1.27)) hide)
-    )
-    (property "Value" "" (id 1) (at 83.185 99.314 0)
-      (effects (font (size 1.27 1.27)))
-    )
-    (property "Footprint" "" (id 2) (at 86.36 97.155 0)
-      (effects (font (size 1.27 1.27)) hide)
-    )
-    (property "Datasheet" "" (id 3) (at 86.36 97.155 0)
-      (effects (font (size 1.27 1.27)) hide)
-    )
+  (symbol (lib_id "power:GND") (at 86.36 102.87 0) (unit 1)
+    (in_bom yes) (on_board yes)
+    (default_instance (reference "U") (unit 1) (value "") (footprint ""))
+    (property "Reference" "U" (id 0) (at 86.36 109.22 0)
+      (effects (font (size 1.27 1.27)) hide)
+    )
+    (property "Value" "" (id 1) (at 83.185 105.029 0)
+      (effects (font (size 1.27 1.27)))
+    )
+    (property "Footprint" "" (id 2) (at 86.36 102.87 0)
+      (effects (font (size 1.27 1.27)) hide)
+    )
+    (property "Datasheet" "" (id 3) (at 86.36 102.87 0)
+      (effects (font (size 1.27 1.27)) hide)
+    )

Commit message: rev.0x6
Parts:
- added FID: Fiducial, symbol Mechanical:Fiducial
Changed lines of the file:
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@@
     (effects (font (size 1.27 1.27)) (justify left bottom))
+  )
+  (symbol (lib_id "Mechanical:Fiducial") (at 195.58 143.51 0) (unit 1)
+    (in_bom yes) (on_board yes) (fields_autoplaced)
+    (default_instance (reference "FID") (unit 1) (value "Fiducial") (footprint ""))
+    (property "Reference" "FID" (id 0) (at 198.12 142.875 0)
+      (effects (font (size 1.27 1.27)) (justify left))
+    )
+    (property "Value" "Fiducial" (id 1) (at 198.12 145.415 0)
+      (effects (font (size 1.27 1.27)) (justify left))
+    )
+    (property "Footprint" "" (id 2) (at 195.58 143.51 0)
+      (effects (font (size 1.27 1.27)) hide)
+    )
+    (property "Datasheet" "~" (id 3) (at 195.58 143.51 0)
+      (effects (font (size 1.27 1.27)) hide)
+    )
   )
   (symbol (lib_id "power:VCC") (at 52.07 129.54 0) (unit 1)
@@
       (reference "#PWR02") (unit 1) (value "VCC") (footprint "")
     )
-    (path "/a12d5f25-796c-439d-8d09-e12e0fd2b9b8"
-      (reference "#PWR02") (unit 1) (value "VCC") (footprint "")
-    )
     (path "/bfc4e6d2-f090-4aed-9faa-0dacd2c9400d"
       (reference "#PWR03") (unit 1) (value "+3.3V") (footprint "")
     )
-    (path "/56756392-a618-4126-b5e1-a59545150644"
-      (reference "#PWR04") (unit 1) (value "GND") (footprint "")
-    )
     (path "/79d967a2-a3fb-4341-a626-f2a28f9639ac"
       (reference "#PWR04") (unit 1) (value "GND") (footprint "")
     )
-    (path "/1c1fcd17-9f67-46ff-8d65-90dacaed7b05"
-      (reference "#PWR05") (unit 1) (value "GND") (footprint "")
-    )
-    (path "/7717233d-248e-4e06-b813-6cfb4b7025b6"
-      (reference "#PWR05") (unit 1) (value "GND") (footprint "")
-    )
     (path "/fb85c0d6-20fe-4277-9b99-e82ff962b53f"
       (reference "#PWR05") (unit 1) (value "GND") (footprint "")
@@
       (reference "#PWR07") (unit 1) (value "+3.3V") (footprint "")
     )
-    (path "/78c52b79-b62a-4123-ad0a-a2f81c23f1a5"
-      (reference "#PWR08") (unit 1) (value "GND") (footprint "")
-    )
-    (path "/83afb465-fdc5-45e8-943d-d073e64deb4d"
-      (reference "#PWR08") (unit 1) (value "GND") (footprint "")
-    )
     (path "/b0f80bfd-5db1-42f9-9ab0-0af67335c0f8"
       (reference "#PWR08") (unit 1) (value "GND") (footprint "")
@@
       (reference "#PWR0102") (unit 1) (value "+3.3V") (footprint "")
     )
+    (path "/1c1fcd17-9f67-46ff-8d65-90dacaed7b05"
+      (reference "#PWR0103") (unit 1) (value "GND") (footprint "")
+    )
+    (path "/7717233d-248e-4e06-b813-6cfb4b7025b6"
+      (reference "#PWR0104") (unit 1) (value "GND") (footprint "")
+    )
+    (path "/78c52b79-b62a-4123-ad0a-a2f81c23f1a5"
+      (reference "#PWR0105") (unit 1) (value "GND") (footprint "")
+    )
+    (path "/83afb465-fdc5-45e8-943d-d073e64deb4d"
+      (reference "#PWR0106") (unit 1) (value "GND") (footprint "")
+    )
+    (path "/56756392-a618-4126-b5e1-a59545150644"
+      (reference "#PWR0107") (unit 1) (value "GND") (footprint "")
+    )
+    (path "/a12d5f25-796c-439d-8d09-e12e0fd2b9b8"
+      (reference "#PWR0108") (unit 1) (value "VCC") (footprint "")
+    )
     (path "/10fad348-e2d5-4988-851d-25e3f509fb5d"
       (reference "C1") (unit 1) (value "1uF") (footprint "Capacitor_SMD:C_0603_1608Metric")
@@
       (reference "D1") (unit 1) (value "DNP") (footprint "LED_SMD:LED_0603_1608Metric")
     )
+    (path "/003076aa-50a2-448f-9bf2-be06998c0f82"
+      (reference "FID1") (unit 1) (value "Fiducial") (footprint "Fiducial:Fiducial_0.5mm_Mask1.5mm")
+    )
     (path "/9c2b882f-dd8b-4c18-b876-9c32757c3278"

Commit message: rev.0x7
Connections:
- net UartRx renamed PA3
- net UartTx renamed PA2
Other:
- moved on the sheet: D, FID, U
