File: placebo.kicad_sch (KiCad schematic)
At the start: 15 parts

Commit message: rev. 0x8
Connections:
- net PB3: no longer U.1
- net PC15: now also U.1
Other:
- moved on the sheet: D, U

Commit message: update BOM
Changed lines of the file:
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@@
       (effects (font (size 1.27 1.27)) (justify left))
     )
-    (property "Value" "" (id 1) (at 86.614 63.246 0)
+    (property "Value" "" (id 1) (at 85.852 63.246 0)
       (effects (font (size 1.27 1.27)) (justify left))
     )
@@
     (in_bom yes) (on_board yes)
     (default_instance (reference "U") (unit 1) (value "") (footprint ""))
-    (property "Reference" "U" (id 0) (at 61.595 136.017 90)
+    (property "Reference" "U" (id 0) (at 63.627 136.017 90)
       (effects (font (size 1.27 1.27)) (justify right))
     )
-    (property "Value" "" (id 1) (at 66.04 136.017 90)
+    (property "Value" "" (id 1) (at 64.516 140.97 90)
       (effects (font (size 1.27 1.27)) (justify right))
     )
@@
       (effects (font (size 1.27 1.27)) hide)
     )
-    (property "Datasheet" "~" (id 3) (at 47.625 131.318 0)
+    (property "Datasheet" "https://www.mouser.com/datasheet/2/348/sml-d12w8w(a)-e-1874513.pdf" (id 3) (at 47.625 131.318 0)
       (effects (font (size 1.27 1.27)) hide)
     )
@@
       (effects (font (size 1.27 1.27)) (justify left))
     )
-    (property "Value" "" (id 1) (at 132.334 63.246 0)
+    (property "Value" "" (id 1) (at 131.318 63.119 0)
       (effects (font (size 1.27 1.27)) (justify left))
     )
@@
     )
     (path "/10fad348-e2d5-4988-851d-25e3f509fb5d"
-      (reference "C1") (unit 1) (value "1uF") (footprint "Capacitor_SMD:C_0603_1608Metric")
+      (reference "C1") (unit 1) (value "10uF") (footprint "Capacitor_SMD:C_0603_1608Metric")
     )
     (path "/ad4e5830-fc9f-4de1-95d7-b549b51196a0"
-      (reference "C2") (unit 1) (value "1uF") (footprint "Capacitor_SMD:C_0603_1608Metric")
+      (reference "C2") (unit 1) (value "10uF") (footprint "Capacitor_SMD:C_0603_1608Metric")
     )
     (path "/ea9ef5aa-2a55-4b4f-b7a1-29bd35e51a5e"
@@
     )
     (path "/88a8f872-f17b-4b37-aeac-a8a5902e3f19"
-      (reference "D1") (unit 1) (value "DNP") (footprint "LED_SMD:LED_0603_1608Metric")
+      (reference "D1") (unit 1) (value "SML-D12W8WT86A") (footprint "LED_SMD:LED_0603_1608Metric")
     )
     (path "/003076aa-50a2-448f-9bf2-be06998c0f82"
@@
     )
     (path "/517410fd-5c0d-4b37-a685-3bd4b7c21b64"
-      (reference "R2") (unit 1) (value "DNP") (footprint "Resistor_SMD:R_0603_1608Metric")
+      (reference "R2") (unit 1) (value "470R") (footprint "Resistor_SMD:R_0603_1608Metric")
     )
     (path "/8f61ea87-2635-46b2-b1be-1f060a135611"

Commit message: update docs
Other:
- moved on the sheet: D, FID, U

Commit message: rev.0x9
Parts:
- C1, C2, C4: renamed from U; value (none) -> 10uF; footprint (none) -> Capacitor_SMD:C_0603_1608Metric
- C3, C5: renamed from U; value (none) -> 100nF; footprint (none) -> Capacitor_SMD:C_0603_1608Metric
- D1: renamed from D; value LED -> SML-D12W8WT86A; footprint (none) -> LED_SMD:LED_0603_1608Metric
- FID1: renamed from FID; footprint (none) -> Fiducial:Fiducial_0.5mm_Mask1.5mm
- J2: renamed from U; value (none) -> TagConnect; footprint (none) -> placebo:Tag-Connect_TC2030-IDC-NL_2x03_P1.27mm_Vertical
- R1: renamed from U; value (none) -> 10K; footprint (none) -> Resistor_SMD:R_0603_1608Metric
- R2: renamed from U; value (none) -> 470R; footprint (none) -> Resistor_SMD:R_0603_1608Metric
- R3, R4: renamed from U; value (none) -> DNP; footprint (none) -> Resistor_SMD:R_0603_1608Metric
- U1: renamed from U; value (none) -> AP7370-33W5-7; footprint (none) -> Package_TO_SOT_SMD:TSOT-23-5_HandSoldering
- U2: renamed from U; value (none) -> STM32G0xxFx; footprint (none) -> Package_SO:TSSOP-20_4.4x6.5mm_P0.65mm
- U3: renamed from U; footprint placebo:PlaceboConnect -> placebo:PlaceboConnect_Cutout
Connections:
- net PA0: now also R2.2
- net PC15: no longer R2.1
- net at D1.1 (K), R3.1: now also R2.1; no longer R2.2
Other:
- moved on the sheet: C3, C4, C5, D1, R1, R2, R3, U2
